File: Hardware/GNSS_Chip_Antenna_Evaluation_Board.brd (EAGLE design)
At the start: 64.8 x 40.6 mm, 68 parts, among them J1 U.FL, J2 U.FL, J3 U.FL, J4 U.FL, J5 U.FL, J6 U.FL, Y2 PUCK, Y3 CUBE, Y4 CHIP, Y5 MOLDED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

Commit message: File rename
Parts:
- moved FRAME1 23.2 mm to (1.27, -15.2)
Other:
- board size 64.8 x 40.6 mm -> 66 x 40.6 mm
- board text added: "V10"
- board text removed: "x01"
Changed lines of the file:
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@@
 <?xml version="1.0" encoding="utf-8"?>
 <!DOCTYPE eagle SYSTEM "eagle.dtd">
-<eagle version="9.2.1">
+<eagle version="9.2.2">
 <drawing>
 <settings>
@@
 <layer number="23" name="tOrigins" color="15" fill="1" visible="yes" active="yes"/>
 <layer number="24" name="bOrigins" color="15" fill="1" visible="yes" active="yes"/>
-<layer number="25" name="tNames" color="7" fill="1" visible="no" active="yes"/>
-<layer number="26" name="bNames" color="7" fill="1" visible="no" active="yes"/>
-<layer number="27" name="tValues" color="7" fill="1" visible="no" active="yes"/>
-<layer number="28" name="bValues" color="7" fill="1" visible="no" active="yes"/>
-<layer number="29" name="tStop" color="2" fill="3" visible="no" active="yes"/>
-<layer number="30" name="bStop" color="5" fill="6" visible="no" active="yes"/>
-<layer number="31" name="tCream" color="7" fill="4" visible="no" active="yes"/>
-<layer number="32" name="bCream" color="7" fill="5" visible="no" active="yes"/>
-<layer number="33" name="tFinish" color="6" fill="3" visible="no" active="yes"/>
-<layer number="34" name="bFinish" color="6" fill="6" visible="no" active="yes"/>
-<layer number="35" name="tGlue" color="7" fill="4" visible="no" active="yes"/>
-<layer number="36" name="bGlue" color="7" fill="5" visible="no" active="yes"/>
-<layer number="37" name="tTest" color="7" fill="1" visible="no" active="yes"/>
-<layer number="38" name="bTest" color="7" fill="1" visible="no" active="yes"/>
-<layer number="39" name="tKeepout" color="4" fill="11" visible="no" active="yes"/>
-<layer number="40" name="bKeepout" color="1" fill="11" visible="no" active="yes"/>
-<layer number="41" name="tRestrict" color="4" fill="10" visible="no" active="yes"/>
-<layer number="42" name="bRestrict" color="1" fill="10" visible="no" active="yes"/>
-<layer number="43" name="vRestrict" color="2" fill="10" visible="no" active="yes"/>
-<layer number="44" name="Drills" color="7" fill="1" visible="no" active="yes"/>
+<layer number="25" name="tNames" color="7" fill="1" visible="yes" active="yes"/>
+<layer number="26" name="bNames" color="7" fill="1" visible="yes" active="yes"/>
+<layer number="27" name="tValues" color="7" fill="1" visible="yes" active="yes"/>
+<layer number="28" name="bValues" color="7" fill="1" visible="yes" active="yes"/>
+<layer number="29" name="tStop" color="2" fill="3" visible="yes" active="yes"/>
+<layer number="30" name="bStop" color="5" fill="6" visible="yes" active="yes"/>
+<layer number="31" name="tCream" color="7" fill="4" visible="yes" active="yes"/>
+<layer number="32" name="bCream" color="7" fill="5" visible="yes" active="yes"/>
+<layer number="33" name="tFinish" color="6" fill="3" visible="yes" active="yes"/>
+<layer number="34" name="bFinish" color="6" fill="6" visible="yes" active="yes"/>
+<layer number="35" name="tGlue" color="7" fill="4" visible="yes" active="yes"/>
+<layer number="36" name="bGlue" color="7" fill="5" visible="yes" active="yes"/>
+<layer number="37" name="tTest" color="7" fill="1" visible="yes" active="yes"/>
+<layer number="38" name="bTest" color="7" fill="1" visible="yes" active="yes"/>
+<layer number="39" name="tKeepout" color="4" fill="11" visible="yes" active="yes"/>
+<layer number="40" name="bKeepout" color="1" fill="11" visible="yes" active="yes"/>
+<layer number="41" name="tRestrict" color="4" fill="10" visible="yes" active="yes"/>
+<layer number="42" name="bRestrict" color="1" fill="10" visible="yes" active="yes"/>
+<layer number="43" name="vRestrict" color="2" fill="10" visible="yes" active="yes"/>
+<layer number="44" name="Drills" color="7" fill="1" visible="yes" active="yes"/>
 <layer number="45" name="Holes" color="7" fill="1" visible="yes" active="yes"/>
-<layer number="46" name="Milling" color="3" fill="1" visible="no" active="yes"/>
-<layer number="47" name="Measures" color="7" fill="1" visible="no" active="yes"/>
-<layer number="48" name="Document" color="7" fill="1" visible="no" active="yes"/>
+<layer number="46" name="Milling" color="3" fill="1" visible="yes" active="yes"/>
+<layer number="47" name="Measures" color="7" fill="1" visible="yes" active="yes"/>
+<layer number="48" name="Document" color="7" fill="1" visible="yes" active="yes"/>
 <layer number="49" name="ReferenceLC" color="13" fill="1" visible="yes" active="yes"/>
-<layer number="50" name="ReferenceLS" color="12" fill="1" visible="no" active="yes"/>
+<layer number="50" name="ReferenceLS" color="12" fill="1" visible="yes" active="yes"/>
 <layer number="51" name="tDocu" color="6" fill="1" visible="yes" active="yes"/>
-<layer number="52" name="bDocu" color="7" fill="1" visible="no" active="yes"/>
+<layer number="52" name="bDocu" color="7" fill="1" visible="yes" active="yes"/>
 <layer number="91" name="Nets" color="2" fill="1" visible="no" active="no"/>
 <layer number="92" name="Busses" color="1" fill="1" visible="no" active="no"/>
@@
 <layer number="13" name="Route13" color="4" fill="5" visible="no" active="no"/>
 <layer number="14" name="Route14" color="1" fill="6" visible="no" active="no"/>
-<layer number="15" name="Route15" color="4" fill="6" visible="no" active="yes"/>
-<layer number="2" name="Route2" color="1" fill="3" visible="no" active="yes"/>
+<layer number="15" name="Route15" color="4" fill="6" visible="no" active="no"/>
+<layer number="2" name="Route2" color="1" fill="3" visible="no" active="no"/>
 <layer number="97" name="Info" color="7" fill="1" visible="no" active="no"/>
 <layer number="98" name="Guide" color="6" fill="1" visible="no" active="no"/>
@@
 <wire x1="0" y1="0" x2="0" y2="35.56" width="0.2032" layer="20"/>
 <text x="0" y="-0.0635" size="0.0254" layer="214" font="vector">D:/SmartProjects/Snc/a4_bn_logo2.bmp</text>
-<text x="20.701" y="0.254" size="1.27" layer="16" font="vector" ratio="20" rot="MR0">x01</text>
+<text x="20.701" y="0.254" size="1.27" layer="16" font="vector" ratio="20" rot="MR0">V10</text>
 <rectangle x1="3.175" y1="22.352" x2="4.572" y2="30.607" layer="43"/>
 <rectangle x1="8.255" y1="23.114" x2="9.906" y2="30.607" layer="43"/>
@@
 <rectangle x1="2.794" y1="12.954" x2="11.938" y2="25.019" layer="43"/>
 <wire x1="25.4" y1="38.1" x2="25.4" y2="-2.54" width="0.1524" layer="20"/>
-<text x="6.35" y="-15.24" size="1.27" layer="51">0.8mm Board Thickness</text>
+<text x="71.12" y="22.86" size="1.27" layer="51">0.8mm Board Thickness</text>
 <text x="25.4" y="-3.81" size="1.27" layer="20" ratio="15" align="center">v-score</text>
 <wire x1="48.26" y1="38.1" x2="48.26" y2="-2.54" width="0.1524" layer="20"/>
 <text x="48.26" y="-3.81" size="1.27" layer="20" ratio="15" align="center">v-score</text>
 <text x="-3.81" y="22.86" size="1.27" layer="20" ratio="15" rot="R270" align="center">v-score</text>
-<wire x1="-1.27" y1="22.86" x2="63.5" y2="22.86" width="0.1524" layer="20"/>
+<wire x1="-2.54" y1="22.86" x2="63.5" y2="22.86" width="0.1524" layer="20"/>
 </plain>
 <attributes>
@@
 <element name="JP9" library="SparkFun" package="FIDUCIAL-1X2" value="FIDUCIAL1X2" x="0.762" y="0.762" smashed="yes"/>
 <element name="U$16" library="SparkFun-Aesthetics" package="OSHW-LOGO-S" value="OSHW-LOGOS" x="19.05" y="3.81" smashed="yes" rot="MR0"/>
-<element name="FRAME1" library="SparkFun-Aesthetics" package="CREATIVE_COMMONS" value="FRAME-LETTER" x="-2.54" y="-38.1" smashed="yes">
-<attribute name="DESIGNER" value="" x="-2.54" y="-38.1" size="1.778" layer="27" font="vector" ratio="15" display="off"/>
-<attribute name="REV" value="" x="-2.54" y="-38.1" size="1.778" layer="27" font="vector" ratio="15" display="off"/>
+<element name="FRAME1" library="SparkFun-Aesthetics" package="CREATIVE_COMMONS" value="FRAME-LETTER" x="1.27" y="-15.24" smashed="yes">
+<attribute name="DESIGNER" value="" x="1.27" y="-15.24" size="1.778" layer="27" font="vector" ratio="15" display="off"/>
+<attribute name="REV" value="" x="1.27" y="-15.24" size="1.778" layer="27" font="vector" ratio="15" display="off"/>
 </element>
 <element name="J1" library="SparkFun-Connectors" package="U.FL" value="U.FL" x="34.29" y="32.004" smashed="yes" rot="R90">

Commit message: Add license, readme, ignore. Add logo. Add GNSS freq table to sch. Touch up sch.
Parts:
- added U$17: (no value), SparkFun-Aesthetics:ORDERING_INSTRUCTIONS
- added U$23: (no value), SparkFun-Aesthetics:SFE_LOGO_NAME_.1
- Y2: device GPS Chip Antennas:TE_PUCK -> GNSS_Chip_Antenna_Evaluation_Board:TE_PUCK
- Y3: device GPS Chip Antennas:MOLEX_GNSS_CUBE -> GNSS_Chip_Antenna_Evaluation_Board:MOLEX_GNSS_CUBE
- Y4: device GPS Chip Antennas:MOLEX_GNSS_CHIP -> GNSS_Chip_Antenna_Evaluation_Board:MOLEX_GNSS_CHIP
- Y5: device GPS Chip Antennas:MLOEX_GNSS_MOLDED -> GNSS_Chip_Antenna_Evaluation_Board:MLOEX_GNSS_MOLDED
- Y6: device GPS Chip Antennas:W3062A -> GNSS_Chip_Antenna_Evaluation_Board:W3062A
- Y7: device GPS Chip Antennas:W3011 -> GNSS_Chip_Antenna_Evaluation_Board:W3011
Changed lines of the file:
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@@
 <setting verticaltext="up"/>
 </settings>
-<grid distance="0.05" unitdist="inch" unit="inch" style="lines" multiple="1" display="yes" altdistance="0.005" altunitdist="inch" altunit="inch"/>
+<grid distance="0.05" unitdist="inch" unit="inch" style="lines" multiple="1" display="yes" altdistance="0.001" altunitdist="inch" altunit="inch"/>
 <layers>
 <layer number="1" name="Top" color="4" fill="1" visible="yes" active="yes"/>
@@
 <text x="0" y="-0.0635" size="0.0254" layer="214" font="vector">D:/SmartProjects/Snc/a4_bn_logo2.bmp</text>
 <text x="20.701" y="0.254" size="1.27" layer="16" font="vector" ratio="20" rot="MR0">V10</text>
-<rectangle x1="3.175" y1="22.352" x2="4.572" y2="30.607" layer="43"/>
-<rectangle x1="8.255" y1="23.114" x2="9.906" y2="30.607" layer="43"/>
-<rectangle x1="50.419" y1="10.795" x2="51.054" y2="11.303" layer="43"/>
-<rectangle x1="52.959" y1="10.668" x2="53.467" y2="11.557" layer="43"/>
-<rectangle x1="13.843" y1="29.337" x2="15.24" y2="31.623" layer="43"/>
-<rectangle x1="2.794" y1="12.954" x2="11.938" y2="25.019" layer="43"/>
 <wire x1="25.4" y1="38.1" x2="25.4" y2="-2.54" width="0.1524" layer="20"/>
-<text x="71.12" y="22.86" size="1.27" layer="51">0.8mm Board Thickness</text>
+<text x="67.31" y="39.37" size="1.27" layer="51">0.8mm Board Thickness</text>
 <text x="25.4" y="-3.81" size="1.27" layer="20" ratio="15" align="center">v-score</text>
 <wire x1="48.26" y1="38.1" x2="48.26" y2="-2.54" width="0.1524" layer="20"/>
@@
 <attribute name="VALUE" x="36.83" y="30.734" size="0.6096" layer="27" font="vector" ratio="20" rot="R90" align="top-left"/>
 </element>
-<element name="Y2" library="GPS Chip Antennas" package="TE_PUCK" value="PUCK" x="12.7" y="13.97" smashed="yes"/>
+<element name="Y2" library="GNSS_Chip_Antenna_Evaluation_Board" package="TE_PUCK" value="PUCK" x="12.7" y="13.97" smashed="yes"/>
 <element name="J2" library="SparkFun-Connectors" package="U.FL" value="U.FL" x="14.478" y="2.667" smashed="yes" rot="R90">
 <attribute name="NAME" x="11.938" y="1.397" size="0.6096" layer="25" font="vector" ratio="20" rot="R90"/>
@@
 <attribute name="VALUE" x="17.018" y="1.397" size="0.6096" layer="27" font="vector" ratio="20" rot="R90" align="top-left"/>
 </element>
-<element name="Y3" library="GPS Chip Antennas" package="MOLEX_GNSS_CUBE" value="CUBE" x="36.83" y="6.35" smashed="yes" rot="R180"/>
+<element name="Y3" library="GNSS_Chip_Antenna_Evaluation_Board" package="MOLEX_GNSS_CUBE" value="CUBE" x="36.83" y="6.35" smashed="yes" rot="R180"/>
 <element name="J3" library="SparkFun-Connectors" package="U.FL" value="U.FL" x="27.94" y="9.779" smashed="yes">
 <attribute name="NAME" x="26.67" y="12.319" size="0.6096" layer="25" font="vector" ratio="20"/>
@@
 <attribute name="VALUE" x="26.67" y="7.239" size="0.6096" layer="27" font="vector" ratio="20" align="top-left"/>
 </element>
-<element name="Y4" library="GPS Chip Antennas" package="MOLEX_GNSS_CHIP" value="CHIP" x="52.07" y="1.143" smashed="yes"/>
+<element name="Y4" library="GNSS_Chip_Antenna_Evaluation_Board" package="MOLEX_GNSS_CHIP" value="CHIP" x="52.07" y="1.143" smashed="yes"/>
 <element name="R1" library="Testing" package="0402-RES" value="0" x="56.007" y="1.651" smashed="yes" rot="R180">
 <attribute name="NAME" x="56.896" y="0.9525" size="0.4064" layer="25" rot="R180"/>
@@
 <attribute name="VALUE" x="55.176" y="5.08" size="0.6096" layer="27" font="vector" ratio="20" rot="R270" align="top-left"/>
 </element>
-<element name="Y5" library="GPS Chip Antennas" package="MLOEX_GNSS_MOLDED" value="MOLDED" x="4.064" y="33.02" smashed="yes" rot="R270"/>
+<element name="Y5" library="GNSS_Chip_Antenna_Evaluation_Board" package="MLOEX_GNSS_MOLDED" value="MOLDED" x="4.064" y="33.02" smashed="yes" rot="R270"/>
 <element name="J5" library="SparkFun-Connectors" package="U.FL" value="U.FL" x="2.159" y="27.686" smashed="yes" rot="R90">
 <attribute name="NAME" x="-0.381" y="26.416" size="0.6096" layer="25" font="vector" ratio="20" rot="R90"/>
@@
 <attribute name="VALUE" x="4.699" y="26.416" size="0.6096" layer="27" font="vector" ratio="20" rot="R90" align="top-left"/>
 </element>
-<element name="Y6" library="GPS Chip Antennas" package="W3062A" value="W3062A" x="58.42" y="30.353" smashed="yes" rot="R270"/>
+<element name="Y6" library="GNSS_Chip_Antenna_Evaluation_Board" package="W3062A" value="W3062A" x="58.42" y="30.353" smashed="yes" rot="R270"/>
 <element name="J6" library="SparkFun-Connectors" package="U.FL" value="U.FL" x="53.34" y="25.4" smashed="yes">
 <attribute name="NAME" x="52.07" y="27.94" size="0.6096" layer="25" font="vector" ratio="20"/>
@@
 <attribute name="VALUE" x="52.07" y="22.86" size="0.6096" layer="27" font="vector" ratio="20" align="top-left"/>
 </element>
-<element name="Y7" library="GPS Chip Antennas" package="W3011" value="W3011" x="40.64" y="34.29" smashed="yes" rot="R180"/>
+<element name="Y7" library="GNSS_Chip_Antenna_Evaluation_Board" package="W3011" value="W3011" x="40.64" y="34.29" smashed="yes" rot="R180"/>
 <element name="U$1" library="SparkFun-Hardware" package="STAND-OFF" value="" x="2.54" y="20.32" smashed="yes">
 <attribute name="NAME" x="2.54" y="22.352" size="0.6096" layer="25" font="vector" ratio="20" align="bottom-center"/>
@@
 <element name="LOGO5" library="SparkFun-Aesthetics" package="SFE_LOGO_FLAME_COPPER_EXPOSED_.1" value="SFE_LOGO_FLAME.1EXP" x="46.228" y="16.51" smashed="yes"/>
 <element name="LOGO6" library="SparkFun-Aesthetics" package="SFE_LOGO_FLAME_COPPER_EXPOSED_.1" value="SFE_LOGO_FLAME.1EXP" x="19.05" y="3.81" smashed="yes"/>
+<element name="U$17" library="SparkFun-Aesthetics" package="ORDERING_INSTRUCTIONS" value="" x="64.77" y="50.8" smashed="yes"/>
+<element name="U$23" library="SparkFun-Aesthetics" package="SFE_LOGO_NAME_.1" value="" x="36.83" y="20.32" smashed="yes"/>
 </elements>
 <signals>
