File: Hardware/GNSS_Chip_Antenna_Evaluation_Board.sch (EAGLE design)
At the start: 19 parts, among them J1 U.FL, J2 U.FL, J3 U.FL, J4 U.FL, J5 U.FL, J6 U.FL, Y2 PUCK, Y3 CUBE, Y4 CHIP, Y5 MOLDED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

Commit message: File rename
Parts:
- added LOGO1, LOGO2, LOGO3, LOGO4, LOGO5, LOGO6: SFE_LOGO_FLAME.1EXP, SparkFun-Aesthetics:SFE_LOGO_FLAME.1EXP
Connections:
- net N$2 renamed FEED3
- net N$3 renamed FEED4
- net N$4 renamed FEED5
- net N$6 renamed FEED2
- net N$7 renamed FEED6
Other:
- note added: "Antenna Type: Chip"
- note added: "Antenna Type: LDS"
- note added: "Antenna Type: Loop"
- note added: "Antenna Type: PIFA"
- note added: "Antenna Type: Raised Puck"
- note added: "Center: 1.575GHz"
- note added: "Gain: 0dBi"
- note added: "Gain: 1.4dBi"
- note added: "Gain: 1dBi"
- note added: "Gain: 2.5dBi"
- note added: "Gain: 2dBi"
- note added: "Gain: 3.4dBi"
- note added: "Part: Molex 1462160001"
- note added: "Part: Molex 1462350001"
- note added: "Part: Molex 2042830001"
- note added: "Part: PulseLarsen W3011"
- note added: "Part: PulseLarsen W3062A"
- note added: "Part: TE 1513634-1"
- note added: "Range: 1.561 - 1.602GHz"
- note added: "Range: 1.565 - 1.585GHz"
- note added: "V10"
- note removed: "X02"
- moved on the sheet: J1, J2, J3, J4, J5, J6, R1, Y2, Y3, Y4, Y5, Y6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

Commit message: Add license, readme, ignore. Add logo. Add GNSS freq table to sch. Touch up sch.
Parts:
- Y2: device GPS Chip Antennas:GPS_CHIP_ANTENNAPUCK -> GNSS_Chip_Antenna_Evaluation_Board:GPS_CHIP_ANTENNAPUCK
- Y3: device GPS Chip Antennas:GPS_CHIP_ANTENNACUBE -> GNSS_Chip_Antenna_Evaluation_Board:GPS_CHIP_ANTENNACUBE
- Y4: device GPS Chip Antennas:GPS_CHIP_ANTENNA2042830001 -> GNSS_Chip_Antenna_Evaluation_Board:GPS_CHIP_ANTENNA2042830001
- Y5: device GPS Chip Antennas:GPS_CHIP_ANTENNA_NOGNDMOLDED -> GNSS_Chip_Antenna_Evaluation_Board:GPS_CHIP_ANTENNA_NOGNDMOLDED
- Y6: device GPS Chip Antennas:GPS_CHIP_ANTENNAW3062A -> GNSS_Chip_Antenna_Evaluation_Board:GPS_CHIP_ANTENNAW3062A
- Y7: device GPS Chip Antennas:GPS_CHIP_ANTENNAW3011 -> GNSS_Chip_Antenna_Evaluation_Board:GPS_CHIP_ANTENNAW3011
Other:
- note added: "BeiDou: 1.561 / 1.575GHz"
- note added: "GLONASS: 1.598-1.609GHz"
- note added: "GNSS L1 Frequencies"
- note added: "GPS: 1.575GHz"
- note added: "Galileo: 1.575GHz"
- note added: "Molex Chip"
- note added: "Molex Cube"
- note added: "Molex Molded"
- note added: "N. Seidle"
- note added: "PulseLarsen W3011"
- note added: "PulseLarsen W3062A"
- note added: "TE Puck"
- moved on the sheet: J1, J2, J3, J5, J6, Y2, Y3, Y5, Y6, Y7

Commit message: Removing lib. Adding test result images.
Parts:
- R1: device Testing:RESISTOR0402-RES -> SparkFun-Resistors:0OHM-0402-1/10W
Changed lines of the file:
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@@
 <?xml version="1.0" encoding="utf-8"?>
 <!DOCTYPE eagle SYSTEM "eagle.dtd">
-<eagle version="9.2.2">
+<eagle version="9.3.0">
 <drawing>
 <settings>
@@
 <part name="GND6" library="SparkFun-PowerSymbols" deviceset="GND" device=""/>
 <part name="Y4" library="GNSS_Chip_Antenna_Evaluation_Board" deviceset="GPS_CHIP_ANTENNA" device="2042830001" value="CHIP"/>
-<part name="R1" library="Testing" deviceset="RESISTOR" device="0402-RES" value="0"/>
+<part name="R1" library="SparkFun-Resistors" deviceset="0OHM" device="-0402-1/10W" value="0"/>
 <part name="J4" library="SparkFun-Connectors" deviceset="U.FL2PIN" device="" value="U.FL"/>
 <part name="GND7" library="SparkFun-PowerSymbols" deviceset="GND" device=""/>

Commit message: Pass review: Change silk. Add dims. Revise a few FPs.
Parts:
- Y2: device GNSS_Chip_Antenna_Evaluation_Board:GPS_CHIP_ANTENNAPUCK -> SparkFun-GPS:GPS_CHIP_ANTENNAPUCK
- Y3: device GNSS_Chip_Antenna_Evaluation_Board:GPS_CHIP_ANTENNACUBE -> SparkFun-GPS:GPS_CHIP_ANTENNACUBE
- Y4: device GNSS_Chip_Antenna_Evaluation_Board:GPS_CHIP_ANTENNA2042830001 -> SparkFun-GPS:GPS_CHIP_ANTENNA2042830001
- Y5: device GNSS_Chip_Antenna_Evaluation_Board:GPS_CHIP_ANTENNA_NOGNDMOLDED -> SparkFun-GPS:GPS_CHIP_ANTENNA_NOGNDMOLDED
- Y6: device GNSS_Chip_Antenna_Evaluation_Board:GPS_CHIP_ANTENNAW3062A -> SparkFun-GPS:GPS_CHIP_ANTENNAW3062A
- Y7: device GNSS_Chip_Antenna_Evaluation_Board:GPS_CHIP_ANTENNAW3011 -> SparkFun-GPS:GPS_CHIP_ANTENNAW3011
Changed lines of the file:
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@@
 <part name="GND1" library="SparkFun-PowerSymbols" deviceset="GND" device=""/>
 <part name="GND2" library="SparkFun-PowerSymbols" deviceset="GND" device=""/>
-<part name="Y2" library="GNSS_Chip_Antenna_Evaluation_Board" deviceset="GPS_CHIP_ANTENNA" device="PUCK" value="PUCK"/>
+<part name="Y2" library="SparkFun-GPS" deviceset="GPS_CHIP_ANTENNA" device="PUCK" value="PUCK"/>
 <part name="J2" library="SparkFun-Connectors" deviceset="U.FL2PIN" device="" value="U.FL"/>
 <part name="GND3" library="SparkFun-PowerSymbols" deviceset="GND" device=""/>
 <part name="GND4" library="SparkFun-PowerSymbols" deviceset="GND" device=""/>
-<part name="Y3" library="GNSS_Chip_Antenna_Evaluation_Board" deviceset="GPS_CHIP_ANTENNA" device="CUBE" value="CUBE"/>
+<part name="Y3" library="SparkFun-GPS" deviceset="GPS_CHIP_ANTENNA" device="CUBE" value="CUBE"/>
 <part name="J3" library="SparkFun-Connectors" deviceset="U.FL2PIN" device="" value="U.FL"/>
 <part name="GND5" library="SparkFun-PowerSymbols" deviceset="GND" device=""/>
 <part name="GND6" library="SparkFun-PowerSymbols" deviceset="GND" device=""/>
-<part name="Y4" library="GNSS_Chip_Antenna_Evaluation_Board" deviceset="GPS_CHIP_ANTENNA" device="2042830001" value="CHIP"/>
+<part name="Y4" library="SparkFun-GPS" deviceset="GPS_CHIP_ANTENNA" device="2042830001" value="CHIP"/>
 <part name="R1" library="SparkFun-Resistors" deviceset="0OHM" device="-0402-1/10W" value="0"/>
 <part name="J4" library="SparkFun-Connectors" deviceset="U.FL2PIN" device="" value="U.FL"/>
 <part name="GND7" library="SparkFun-PowerSymbols" deviceset="GND" device=""/>
 <part name="GND8" library="SparkFun-PowerSymbols" deviceset="GND" device=""/>
-<part name="Y5" library="GNSS_Chip_Antenna_Evaluation_Board" deviceset="GPS_CHIP_ANTENNA_NOGND" device="MOLDED" value="MOLDED"/>
+<part name="Y5" library="SparkFun-GPS" deviceset="GPS_CHIP_ANTENNA_NOGND" device="MOLDED" value="MOLDED"/>
 <part name="J5" library="SparkFun-Connectors" deviceset="U.FL2PIN" device="" value="U.FL"/>
 <part name="GND9" library="SparkFun-PowerSymbols" deviceset="GND" device=""/>
-<part name="Y6" library="GNSS_Chip_Antenna_Evaluation_Board" deviceset="GPS_CHIP_ANTENNA" device="W3062A" value="W3062A"/>
+<part name="Y6" library="SparkFun-GPS" deviceset="GPS_CHIP_ANTENNA" device="W3062A" value="W3062A"/>
 <part name="J6" library="SparkFun-Connectors" deviceset="U.FL2PIN" device="" value="U.FL"/>
 <part name="GND10" library="SparkFun-PowerSymbols" deviceset="GND" device=""/>
 <part name="GND11" library="SparkFun-PowerSymbols" deviceset="GND" device=""/>
-<part name="Y7" library="GNSS_Chip_Antenna_Evaluation_Board" deviceset="GPS_CHIP_ANTENNA" device="W3011" value="W3011"/>
+<part name="Y7" library="SparkFun-GPS" deviceset="GPS_CHIP_ANTENNA" device="W3011" value="W3011"/>
 <part name="LOGO1" library="SparkFun-Aesthetics" deviceset="SFE_LOGO_FLAME" device=".1EXP"/>
 <part name="LOGO2" library="SparkFun-Aesthetics" deviceset="SFE_LOGO_FLAME" device=".1EXP"/>
